File: Hardware/Production/SparkFun_GNSS_NEO-M9N-Panel.brd (EAGLE design)
At the start: 135.2 x 149.5 mm, 468 parts, among them J1 MICROMOD_STANDARD, J10 MICROMOD_STANDARD, J12 Bus Selection, J14 MICROMOD_STANDARD, J16 Bus Selection, J18 MICROMOD_STANDARD, J20 Bus Selection, J22 MICROMOD_STANDARD, J24 Bus Selection, J4 Bus Selection, J6 MICROMOD_STANDARD, J8 Bus Selection, U1 U-BLOX_NEO-M9N, U10 U-BLOX_NEO-M9N, U11 EEPROM, U12 74HC1G04, U13 3.3V, U14 U-BLOX_NEO-M9N, U15 EEPROM, U16 74HC1G04, U17 3.3V, U18 U-BLOX_NEO-M9N, U19 EEPROM, U2 3.3V, U20 74HC1G04, U21 3.3V, U22 U-BLOX_NEO-M9N, U23 EEPROM, U24 74HC1G04, U3 EEPROM, U4 74HC1G04, U5 3.3V, U6 U-BLOX_NEO-M9N, U7 EEPROM, U8 74HC1G04, U9 3.3V

Commit message: Updated production files to v12
Parts:
- B1, B2, B3, B4, B5, B6: device SparkFun-Batteries:ML414H_IV01E -> SparkFun-Batteries:MS421R_IV03E
- E1, E2, E3, E4, E5, E6: value ANTENNA-SMA-GROUNDEDEDGE_SMA_THIN -> U.FL; device SparkFun-RF:SMA-EDGE -> SparkFun-Connectors:U.FL
- R17, R18, R33, R34, R49, R50, R65, R66, R7, R8, R81, R82: value 4.7k -> 2.2k
- R19, R35, R5, R51, R67, R83: value 1k -> 3.3k
- moved U$140 8.64 mm to (109.0, 80.8)
- moved U$62 8.64 mm to (83.3, 55.4)
- moved U$88 8.64 mm to (31.9, 80.8)
- moved U$14 8.64 mm to (6.17, 55.4)
- moved U$36 8.64 mm to (44.7, 55.4)
- moved U$114 8.64 mm to (70.4, 80.8)
- moved E4 7.06 mm to (27.9, 80.5), turned to 90 degrees
- moved E5 7.06 mm to (66.5, 80.5), turned to 90 degrees
- moved E6 7.06 mm to (105.1, 80.5), turned to 90 degrees
- moved E1 7.06 mm to (10.1, 55.7), turned to 270 degrees
- moved E2 7.06 mm to (48.7, 55.7), turned to 270 degrees
- moved E3 7.06 mm to (87.2, 55.7), turned to 270 degrees
- moved U$109 4.60 mm to (69.1, 78.6)
- moved U$135 4.60 mm to (107.7, 78.6)
- moved U$83 4.60 mm to (30.6, 78.6)
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Connections:
- net GND: now also E1.1, E1.2; no longer E1.GND@0, E1.GND@1, E1.GND@2, E1.GND@3
- net GND1: now also E2.1, E2.2; no longer E2.GND@0, E2.GND@1, E2.GND@2, E2.GND@3
- net GND2: now also E3.1, E3.2; no longer E3.GND@0, E3.GND@1, E3.GND@2, E3.GND@3
- net GND3: now also E4.1, E4.2; no longer E4.GND@0, E4.GND@1, E4.GND@2, E4.GND@3
- net GND4: now also E5.1, E5.2; no longer E5.GND@0, E5.GND@1, E5.GND@2, E5.GND@3
- net GND5: now also E6.1, E6.2; no longer E6.GND@0, E6.GND@1, E6.GND@2, E6.GND@3
- net GPS_ANT1: now also E1.FEED; no longer E1.SIG
- net GPS_ANT2: now also E2.FEED; no longer E2.SIG
- net GPS_ANT3: now also E3.FEED; no longer E3.SIG
- net GPS_ANT4: now also E4.FEED; no longer E4.SIG
- net GPS_ANT5: now also E5.FEED; no longer E5.SIG
- net GPS_ANT6: now also E6.FEED; no longer E6.SIG
Routing:
- net 3.3V5: track 147.1 -> 148.2 mm
- net 3.3V4: track 147.1 -> 148.2 mm
- net 3.3V3: track 147.1 -> 148.2 mm
- net 3.3V2: track 147.1 -> 148.2 mm
- net 3.3V1: track 147.1 -> 148.2 mm
- net 3.3V: track 147.1 -> 148.2 mm
- net GND5: vias 204 -> 205
- net GND4: vias 204 -> 205
- net GND3: vias 204 -> 205
- net GND2: vias 204 -> 205
- net GND1: vias 204 -> 205
- net GND: vias 204 -> 205
Other:
- board text added: "v12"
- board text removed: "v11"

Commit message: Revised panel
Parts:
- J1, J10, J14, J18, J22, J6: value MICROMOD_STANDARD -> MICROMOD_FUNCTION_STANDARD; device SparkFun-MicroMod-Function:M.2-CARD-E-22_FUNCTION_STANDARD -> SparkFun-MicroMod:M.2-CARD-E-22_FUNCTION_STANDARD
- U1, U10, U14, U18, U22, U6: device SparkFun-GPS:NEO-M9N/M8T/M8U -> SparkFun-GPS:NEO-M9N/M8T/M8U/D9S
- moved E$3 1.68 mm to (116.1, 129.9)
- moved E$4 1.68 mm to (116.1, 129.9)
- moved C21 1.42 mm to (101.1, 27.7)
- moved D7 1.42 mm to (103.5, 25.8)
- moved FB3 1.42 mm to (86.4, 48.4)
- moved LOGO6 1.42 mm to (111.3, 10.2)
- moved R35 1.42 mm to (103.5, 24.2)
- moved R39 1.42 mm to (104.0, 51.9)
- moved R42 1.42 mm to (81.3, 8.66)
- moved R43 1.42 mm to (96.4, 26.2)
- moved R44 1.42 mm to (78.6, 32.0)
- moved R45 1.42 mm to (99.3, 55.4)
- moved TP3 1.42 mm to (110.6, 22.8)
- moved U$54 1.42 mm to (93.0, 60.4)
- moved U$55 1.42 mm to (84.4, 41.2)
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Other:
- board size 135.2 x 149.5 mm -> 133.6 x 149.5 mm
