File: Hardware/SparkFun_GNSS_NEO-M9N.sch (EAGLE design)
At the start: 55 parts, among them J1 MICROMOD_STANDARD, J4 Bus Selection, U1 U-BLOX_NEO-M9N, U2 3.3V, U3 EEPROM, U4 74HC1G04

Commit message: Replaces old ML414H reflowable with new MS421R
Parts:
- B1: device SparkFun-Batteries:ML414H_IV01E_BATTERY -> SparkFun-Batteries:RELOWABLE_BATTERY_MS421R
Other:
- note added: "u.FL Connector"
- note removed: "SMA Connector"
Changed lines of the file:
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@@
 <part name="GND3" library="SparkFun-PowerSymbols" deviceset="GND" device=""/>
 <part name="C3" library="SparkFun-Capacitors" deviceset="1.0UF" device="-0603-16V-10%" value="1.0uF"/>
-<part name="B1" library="SparkFun-Batteries" deviceset="ML414H_IV01E_BATTERY" device="" value="6.8MM_COIN_CELL"/>
+<part name="B1" library="SparkFun-Batteries" deviceset="RELOWABLE_BATTERY" device="_MS421R" value="6.8MM_COIN_CELL"/>
 <part name="GND5" library="SparkFun-PowerSymbols" deviceset="GND" device=""/>
 <part name="GND10" library="SparkFun-PowerSymbols" deviceset="GND" device=""/>
@@
 <text x="170.18" y="86.36" size="2.54" layer="94" font="vector" align="center">Hot Start Battery</text>
 <text x="73.66" y="269.24" size="2.54" layer="94" font="vector" align="center">GPS: u-Blox NEO-M9N </text>
-<text x="231.902" y="86.614" size="2.54" layer="94" font="vector" align="center">SMA Connector</text>
+<text x="231.902" y="86.614" size="2.54" layer="94" font="vector" align="center">u.FL Connector</text>
 <text x="58.42" y="241.3" size="1.27" layer="97" font="vector">VCC Range: 2.7V - 3.3V</text>
 <wire x1="284.48" y1="8.89" x2="284.48" y2="17.78" width="0.2032" layer="97" style="dashdot"/>
@@
 <text x="60.96" y="76.2" size="2.54" layer="94" font="vector" align="center">EEPROM</text>
 <text x="363.22" y="271.78" size="2.54" layer="94" font="vector" align="center">Voltage Regulation: AP2112K</text>
-<text x="226.06" y="60.96" size="1.778" layer="97" font="vector">L1 Antenna</text>
+<text x="223.52" y="81.28" size="1.778" layer="97" font="vector">L1 Antenna</text>
 <wire x1="142.24" y1="279.4" x2="142.24" y2="198.12" width="0.2032" layer="97" style="longdash"/>
 <wire x1="142.24" y1="198.12" x2="142.24" y2="144.78" width="0.2032" layer="97" style="longdash"/>

Commit message: Uses the updated function board outline
Parts:
- J1: value MICROMOD_STANDARD -> MICROMOD_FUNCTION_STANDARD; device SparkFun-MicroMod-Function:MICROMOD_STANDARD -> SparkFun-MicroMod:MICROMOD_FUNCTION_STANDARD
Changed lines of the file:
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@@
 <part name="FD4" library="SparkFun-Aesthetics" deviceset="FIDUCIAL" device="1X2" value="FIDUCIAL1X2"/>
 <part name="LOGO1" library="SparkFun-Aesthetics" deviceset="SPECIAL_INSTRUCTIONS" device="-ORDERING"/>
-<part name="J1" library="SparkFun-MicroMod-Function" deviceset="MICROMOD" device="_STANDARD" value="MICROMOD_STANDARD"/>
+<part name="J1" library="SparkFun-MicroMod" deviceset="MICROMOD_FUNCTION" device="_STANDARD" value="MICROMOD_FUNCTION_STANDARD"/>
 <part name="GND4" library="SparkFun-PowerSymbols" deviceset="GND" device=""/>
 <part name="GND6" library="SparkFun-PowerSymbols" deviceset="GND" device=""/>

Commit message: Corrects typo on "u-blox" in schematic
Other:
- note added: "GPS: u-blox NEO-M9N"
- note removed: "GPS: u-Blox NEO-M9N"
Changed lines of the file:
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@@
 <text x="297.18" y="88.9" size="2.54" layer="94" font="vector" align="center">LEDs and Jumpers</text>
 <text x="170.18" y="86.36" size="2.54" layer="94" font="vector" align="center">Hot Start Battery</text>
-<text x="73.66" y="269.24" size="2.54" layer="94" font="vector" align="center">GPS: u-Blox NEO-M9N </text>
+<text x="73.66" y="269.24" size="2.54" layer="94" font="vector" align="center">GPS: u-blox NEO-M9N </text>
 <text x="231.902" y="86.614" size="2.54" layer="94" font="vector" align="center">u.FL Connector</text>
 <text x="58.42" y="241.3" size="1.27" layer="97" font="vector">VCC Range: 2.7V - 3.3V</text>
